Commit message: x3plus' gripper took me a lot of time and tokens. but finally it displays properly in isaac sim. good news

File: src/monty_demo/x3plus_isaac/urdf/x3plus_isaac.urdf (robot description, URDF)
Before this commit: robot x3plus_isaac, 17 links, 16 joints
Joints:
- joint arm_joint1: limit lower=-1.5708 upper=1.5708 effort=100 velocity=1 -> lower=-1.5708 upper=1.5708 effort=300 velocity=1
- joint arm_joint2: limit lower=-1.5708 upper=1.5708 effort=100 velocity=1 -> lower=-1.5708 upper=1.5708 effort=300 velocity=1
- joint arm_joint3: limit lower=-1.5708 upper=1.5708 effort=100 velocity=1 -> lower=-1.5708 upper=1.5708 effort=300 velocity=1
- joint arm_joint4: limit lower=-1.5708 upper=1.5708 effort=100 velocity=1 -> lower=-1.5708 upper=1.5708 effort=300 velocity=1
- joint arm_joint5: limit lower=-1.5708 upper=3.14159 effort=100 velocity=1 -> lower=-1.5708 upper=3.14159 effort=300 velocity=1
- joint grip_joint: limit lower=-1.54 upper=0 effort=100 velocity=1 -> lower=-1.54 upper=0 effort=300 velocity=1
