Commit message: the robot moved in the isaac sim.

File: src/monty_demo/x3plus_robot/urdf/ros2_control_topic.xacro (robot description, xacro)
@@ -4,5 +4,8 @@
      Include from x3plus.urdf.xacro.
      NOTE: The <robot> wrapper is required so xacro:include preserves the <ros2_control>
-     element in the output (xacro strips the root element of included files). -->
+     element in the output (xacro strips the root element of included files).
+     Mimic joints (rlink/llink) are NOT listed here; they are computed by the bridge
+     nodes and the URDF <mimic> tags handle TF. Jazzy ros2_control rejects mimic
+     joints that appear in ros2_control when the URDF also has <mimic> attributes. -->
 <robot xmlns:xacro="http://www.ros.org/wiki/xacro">
   <ros2_control name="x3plus" type="system">
@@ -55,29 +58,4 @@
       <state_interface name="position"><param name="initial_value">-0.77</param></state_interface>
     </joint>
-    <joint name="rlink_joint2">
-      <param name="mimic">grip_joint</param>
-      <param name="multiplier">-1</param>
-      <state_interface name="position"><param name="initial_value">0.77</param></state_interface>
-    </joint>
-    <joint name="rlink_joint3">
-      <param name="mimic">grip_joint</param>
-      <param name="multiplier">1</param>
-      <state_interface name="position"><param name="initial_value">-0.77</param></state_interface>
-    </joint>
-    <joint name="llink_joint1">
-      <param name="mimic">grip_joint</param>
-      <param name="multiplier">-1</param>
-      <state_interface name="position"><param name="initial_value">0.77</param></state_interface>
-    </joint>
-    <joint name="llink_joint2">
-      <param name="mimic">grip_joint</param>
-      <param name="multiplier">1</param>
-      <state_interface name="position"><param name="initial_value">-0.77</param></state_interface>
-    </joint>
-    <joint name="llink_joint3">
-      <param name="mimic">grip_joint</param>
-      <param name="multiplier">-1</param>
-      <state_interface name="position"><param name="initial_value">0.77</param></state_interface>
-    </joint>
   </ros2_control>
 </robot>
