Commit message: the gripper is ok. yes!

File: docker_all/shared/x3plus_isaac/urdf/x3plus_isaac.urdf (robot description, URDF)
Before this commit: robot x3plus_isaac, 17 links, 16 joints
Joints:
- joint llink_joint1: mimic (none) -> joint=grip_joint multiplier=-1 offset=0
- joint llink_joint2: mimic (none) -> joint=grip_joint multiplier=1 offset=0
- joint llink_joint3: mimic (none) -> joint=grip_joint multiplier=-1 offset=0
- joint rlink_joint2: mimic (none) -> joint=grip_joint multiplier=-1 offset=0
- joint rlink_joint3: mimic (none) -> joint=grip_joint multiplier=1 offset=0
