Commit message: Add pick-and-place service, file logging, shared init positions, and safety rules
New nodes/scripts:
- x3plus_pick_place: pick/place service orchestrator (gripper + planner)
- pick_place_test: 100-point pick-and-place validation test
- log_utils: rotating file logger (5 MB × 3 backups to /tmp)
- sim_up.sh: convenience script for simulation mode
- init_positions.yaml: single-source home position config

Planner (x3plus_5dof_planner):
- plan_position_orient, plan_straight_line, and set_gripper services
- Dry-run lockout at multiple levels (defense-in-depth)
- File logging for all safety-critical decisions

ZMQ bridge:
- File logging with throttled state dumps
- Watchdog: lockout on 5+ consecutive command/state failures

Isaac bridge:
- Remove ad-hoc debug logging, use shared init positions from YAML

Infra:
- Dockerfiles bake in init_positions.yaml as fallback
- Cursor rules: logging-discipline, robot-motion-safety, x3plus-gripper-geometry

Made-with: Cursor

File: docker_all/components/ros2_comp/app/monty_demo/x3plus_robot/urdf/ros2_control_topic.xacro (robot description, xacro)
@@ -7,6 +7,16 @@
      Mimic joints (rlink/llink) are NOT listed here; they are computed by the bridge
      nodes and the URDF <mimic> tags handle TF. Jazzy ros2_control rejects mimic
-     joints that appear in ros2_control when the URDF also has <mimic> attributes. -->
+     joints that appear in ros2_control when the URDF also has <mimic> attributes.
+     initial_value: bootstrap fallback for ros2_control before the first
+     /x3plus/joint_states message arrives.  Source of truth:
+       shared/x3plus_config/init_positions.yaml
+     Values are passed as xacro args at Docker build time. -->
 <robot xmlns:xacro="http://www.ros.org/wiki/xacro">
+  <xacro:arg name="init_j1"   default="0.0"/>
+  <xacro:arg name="init_j2"   default="-1.0"/>
+  <xacro:arg name="init_j3"   default="-0.8"/>
+  <xacro:arg name="init_j4"   default="-1.3416"/>
+  <xacro:arg name="init_j5"   default="0.0"/>
+  <xacro:arg name="init_grip" default="-0.77"/>
   <ros2_control name="x3plus" type="system">
     <hardware>
@@ -21,5 +31,5 @@
         <param name="max">1.5708</param>
       </command_interface>
-      <state_interface name="position"><param name="initial_value">0.0</param></state_interface>
+      <state_interface name="position"><param name="initial_value">$(arg init_j1)</param></state_interface>
     </joint>
     <joint name="arm_joint2">
@@ -28,5 +38,5 @@
         <param name="max">1.5708</param>
       </command_interface>
-      <state_interface name="position"><param name="initial_value">0.0</param></state_interface>
+      <state_interface name="position"><param name="initial_value">$(arg init_j2)</param></state_interface>
     </joint>
     <joint name="arm_joint3">
@@ -35,5 +45,5 @@
         <param name="max">1.5708</param>
       </command_interface>
-      <state_interface name="position"><param name="initial_value">0.0</param></state_interface>
+      <state_interface name="position"><param name="initial_value">$(arg init_j3)</param></state_interface>
     </joint>
     <joint name="arm_joint4">
@@ -42,5 +52,5 @@
         <param name="max">1.5708</param>
       </command_interface>
-      <state_interface name="position"><param name="initial_value">0.0</param></state_interface>
+      <state_interface name="position"><param name="initial_value">$(arg init_j4)</param></state_interface>
     </joint>
     <joint name="arm_joint5">
@@ -49,5 +59,5 @@
         <param name="max">3.14159</param>
       </command_interface>
-      <state_interface name="position"><param name="initial_value">0.0</param></state_interface>
+      <state_interface name="position"><param name="initial_value">$(arg init_j5)</param></state_interface>
     </joint>
     <joint name="grip_joint">
@@ -56,5 +66,5 @@
         <param name="max">0</param>
       </command_interface>
-      <state_interface name="position"><param name="initial_value">-0.77</param></state_interface>
+      <state_interface name="position"><param name="initial_value">$(arg init_grip)</param></state_interface>
     </joint>
   </ros2_control>
