Commit message: Add MoveIt2 config, 5DOF planner, and clean up duplicated meshes/URDFs
Remove duplicated STL meshes and static URDFs in favor of shared location
and xacro-generated URDFs. Add MoveIt2 configuration (SRDF, kinematics,
joint limits, OMPL planning, controllers), x3plus 5DOF arm planner,
MoveIt launch file, Isaac URDF generation script, and workspace
reachability analysis tools. Update Dockerfiles and compose accordingly.

Made-with: Cursor

File: docker_all/components/ros2_comp/app/monty_demo/x3plus_robot/urdf/x3plus.urdf.xacro (robot description, xacro)
@@ -1,5 +1,13 @@
 <?xml version="1.0" encoding="utf-8"?>
-<robot name="x3plus" xmlns:xacro="http://www.ros.org/wiki/xacro">
-    <xacro:property name="include_ros2_control" value="true"/>
+<!-- Single source of truth for the X3plus robot description.
+     Generate the plain Isaac Sim URDF via:
+       xacro x3plus.urdf.xacro include_ros2_control:=false mesh_prefix:=../meshes robot_name:=x3plus_isaac
+     ROS2 bringup uses the defaults (package://monty_demo/meshes, ros2_control enabled). -->
+<robot name="$(arg robot_name)" xmlns:xacro="http://www.ros.org/wiki/xacro">
+    <xacro:arg name="robot_name" default="x3plus"/>
+    <xacro:arg name="mesh_prefix" default="package://monty_demo/meshes"/>
+    <xacro:arg name="include_ros2_control" default="true"/>
+    <xacro:property name="mesh_prefix" value="$(arg mesh_prefix)"/>
+    <xacro:property name="include_ros2_control" value="$(arg include_ros2_control)"/>
     <link name="base_footprint"/>
     <link name="imu_link"/>
@@ -19,14 +27,14 @@
             <origin xyz="0 0 0" rpy="0 0 0"/>
             <geometry>
-                <mesh filename="package://monty_demo/meshes/X3plus/visual/base_link.STL"/>
-            </geometry>
-            <material name="">
-                <color rgba="0 0.7 0 1"/>
-            </material>
-        </visual>
-        <collision>
-            <origin xyz="0 0 0" rpy="0 0 0"/>
-            <geometry>
-                <mesh filename="package://monty_demo/meshes/X3plus/collision/base_link.STL"/>
+                <mesh filename="${mesh_prefix}/X3plus/visual/base_link.STL"/>
+            </geometry>
+            <material name="">
+                <color rgba="0 0.7 0 1"/>
+            </material>
+        </visual>
+        <collision>
+            <origin xyz="0 0 0" rpy="0 0 0"/>
+            <geometry>
+                <mesh filename="${mesh_prefix}/X3plus/collision/base_link.STL"/>
             </geometry>
         </collision>
@@ -57,5 +65,5 @@
             <origin xyz="0 0 0" rpy="0 0 0"/>
             <geometry>
-                <mesh filename="package://monty_demo/meshes/sensor/visual/camera_link.STL"/>
+                <mesh filename="${mesh_prefix}/sensor/visual/camera_link.STL"/>
             </geometry>
             <material name="">
@@ -66,5 +74,5 @@
             <origin xyz="0 0 0" rpy="0 0 0"/>
             <geometry>
-                <mesh filename="package://monty_demo/meshes/sensor/collision/camera_link.STL"/>
+                <mesh filename="${mesh_prefix}/sensor/collision/camera_link.STL"/>
             </geometry>
         </collision>
@@ -90,5 +98,5 @@
             <origin xyz="0 0 0" rpy="0 0 0"/>
             <geometry>
-                <mesh filename="package://monty_demo/meshes/sensor/visual/laser_link.STL"/>
+                <mesh filename="${mesh_prefix}/sensor/visual/laser_link.STL"/>
             </geometry>
             <material name="">
@@ -99,5 +107,5 @@
             <origin xyz="0 0 0" rpy="0 0 0"/>
             <geometry>
-                <mesh filename="package://monty_demo/meshes/sensor/collision/laser_link.STL"/>
+                <mesh filename="${mesh_prefix}/sensor/collision/laser_link.STL"/>
             </geometry>
         </collision>
@@ -123,5 +131,5 @@
             <origin xyz="0 0 0" rpy="0 0 0"/>
             <geometry>
-                <mesh filename="package://monty_demo/meshes/X3plus/visual/arm_link1.STL"/>
+                <mesh filename="${mesh_prefix}/X3plus/visual/arm_link1.STL"/>
             </geometry>
             <material name="">
@@ -132,5 +140,5 @@
             <origin xyz="0 0 0" rpy="0 0 0"/>
             <geometry>
-                <mesh filename="package://monty_demo/meshes/X3plus/collision/arm_link1.STL"/>
+                <mesh filename="${mesh_prefix}/X3plus/collision/arm_link1.STL"/>
             </geometry>
         </collision>
@@ -158,14 +166,14 @@
             <origin xyz="0 0 0" rpy="0 0 0"/>
             <geometry>
-                <mesh filename="package://monty_demo/meshes/X3plus/visual/arm_link2.STL"/>
-            </geometry>
-            <material name="">
-                <color rgba="0 0.7 0 1"/>
-            </material>
-        </visual>
-        <collision>
-            <origin xyz="0 0 0" rpy="0 0 0"/>
-            <geometry>
-                <mesh filename="package://monty_demo/meshes/X3plus/collision/arm_link2.STL"/>
+                <mesh filename="${mesh_prefix}/X3plus/visual/arm_link2.STL"/>
+            </geometry>
+            <material name="">
+                <color rgba="0 0.7 0 1"/>
+            </material>
+        </visual>
+        <collision>
+            <origin xyz="0 0 0" rpy="0 0 0"/>
+            <geometry>
+                <mesh filename="${mesh_prefix}/X3plus/collision/arm_link2.STL"/>
             </geometry>
         </collision>
@@ -193,5 +201,5 @@
             <origin xyz="0 0 0" rpy="0 0 0"/>
             <geometry>
-                <mesh filename="package://monty_demo/meshes/X3plus/visual/arm_link3.STL"/>
+                <mesh filename="${mesh_prefix}/X3plus/visual/arm_link3.STL"/>
             </geometry>
             <material name="">
@@ -202,5 +210,5 @@
             <origin xyz="0 0 0" rpy="0 0 0"/>
             <geometry>
-                <mesh filename="package://monty_demo/meshes/X3plus/collision/arm_link3.STL"/>
+                <mesh filename="${mesh_prefix}/X3plus/collision/arm_link3.STL"/>
             </geometry>
         </collision>
@@ -228,14 +236,14 @@
             <origin xyz="0 0 0" rpy="0 0 0"/>
             <geometry>
-                <mesh filename="package://monty_demo/meshes/X3plus/visual/arm_link4.STL"/>
-            </geometry>
-            <material name="">
-                <color rgba="0 0.7 0 1"/>
-            </material>
-        </visual>
-        <collision>
-            <origin xyz="0 0 0" rpy="0 0 0"/>
-            <geometry>
-                <mesh filename="package://monty_demo/meshes/X3plus/collision/arm_link4.STL"/>
+                <mesh filename="${mesh_prefix}/X3plus/visual/arm_link4.STL"/>
+            </geometry>
+            <material name="">
+                <color rgba="0 0.7 0 1"/>
+            </material>
+        </visual>
+        <collision>
+            <origin xyz="0 0 0" rpy="0 0 0"/>
+            <geometry>
+                <mesh filename="${mesh_prefix}/X3plus/collision/arm_link4.STL"/>
             </geometry>
         </collision>
@@ -263,5 +271,5 @@
             <origin xyz="0 0 0" rpy="0 0 0"/>
             <geometry>
-                <mesh filename="package://monty_demo/meshes/X3plus/visual/arm_link5.STL"/>
+                <mesh filename="${mesh_prefix}/X3plus/visual/arm_link5.STL"/>
             </geometry>
             <material name="">
@@ -272,5 +280,5 @@
             <origin xyz="0 0 0" rpy="0 0 0"/>
             <geometry>
-                <mesh filename="package://monty_demo/meshes/X3plus/collision/arm_link5.STL"/>
+                <mesh filename="${mesh_prefix}/X3plus/collision/arm_link5.STL"/>
             </geometry>
         </collision>
@@ -298,14 +306,14 @@
             <origin xyz="0 0 0" rpy="0 0 0"/>
             <geometry>
-                <mesh filename="package://monty_demo/meshes/X3plus/visual/rlink1.STL"/>
-            </geometry>
-            <material name="">
-                <color rgba="0 0.7 0 1"/>
-            </material>
-        </visual>
-        <collision>
-            <origin xyz="0 0 0" rpy="0 0 0"/>
-            <geometry>
-                <mesh filename="package://monty_demo/meshes/X3plus/visual/rlink1.STL"/>
+                <mesh filename="${mesh_prefix}/X3plus/visual/rlink1.STL"/>
+            </geometry>
+            <material name="">
+                <color rgba="0 0.7 0 1"/>
+            </material>
+        </visual>
+        <collision>
+            <origin xyz="0 0 0" rpy="0 0 0"/>
+            <geometry>
+                <mesh filename="${mesh_prefix}/X3plus/visual/rlink1.STL"/>
             </geometry>
         </collision>
@@ -333,14 +341,14 @@
             <origin xyz="0 0 0" rpy="0 0 0"/>
             <geometry>
-                <mesh filename="package://monty_demo/meshes/X3plus/visual/rlink2.STL"/>
-            </geometry>
-            <material name="">
-                <color rgba="0 0.7 0 1"/>
-            </material>
-        </visual>
-        <collision>
-            <origin xyz="0 0 0" rpy="0 0 0"/>
-            <geometry>
-                <mesh filename="package://monty_demo/meshes/X3plus/visual/rlink2.STL"/>
+                <mesh filename="${mesh_prefix}/X3plus/visual/rlink2.STL"/>
+            </geometry>
+            <material name="">
+                <color rgba="0 0.7 0 1"/>
+            </material>
+        </visual>
+        <collision>
+            <origin xyz="0 0 0" rpy="0 0 0"/>
+            <geometry>
+                <mesh filename="${mesh_prefix}/X3plus/visual/rlink2.STL"/>
             </geometry>
         </collision>
@@ -368,14 +376,14 @@
             <origin xyz="0 0 0" rpy="0 0 0"/>
             <geometry>
-                <mesh filename="package://monty_demo/meshes/X3plus/visual/rlink3.STL"/>
-            </geometry>
-            <material name="">
-                <color rgba="0 0.7 0 1"/>
-            </material>
-        </visual>
-        <collision>
-            <origin xyz="0 0 0" rpy="0 0 0"/>
-            <geometry>
-                <mesh filename="package://monty_demo/meshes/X3plus/visual/rlink3.STL"/>
+                <mesh filename="${mesh_prefix}/X3plus/visual/rlink3.STL"/>
+            </geometry>
+            <material name="">
+                <color rgba="0 0.7 0 1"/>
+            </material>
+        </visual>
+        <collision>
+            <origin xyz="0 0 0" rpy="0 0 0"/>
+            <geometry>
+                <mesh filename="${mesh_prefix}/X3plus/visual/rlink3.STL"/>
             </geometry>
         </collision>
@@ -403,14 +411,14 @@
             <origin xyz="0 0 0" rpy="0 0 0"/>
             <geometry>
-                <mesh filename="package://monty_demo/meshes/X3plus/visual/llink1.STL"/>
-            </geometry>
-            <material name="">
-                <color rgba="0 0.7 0 1"/>
-            </material>
-        </visual>
-        <collision>
-            <origin xyz="0 0 0" rpy="0 0 0"/>
-            <geometry>
-                <mesh filename="package://monty_demo/meshes/X3plus/visual/llink1.STL"/>
+                <mesh filename="${mesh_prefix}/X3plus/visual/llink1.STL"/>
+            </geometry>
+            <material name="">
+                <color rgba="0 0.7 0 1"/>
+            </material>
+        </visual>
+        <collision>
+            <origin xyz="0 0 0" rpy="0 0 0"/>
+            <geometry>
+                <mesh filename="${mesh_prefix}/X3plus/visual/llink1.STL"/>
             </geometry>
         </collision>
@@ -433,14 +441,14 @@
             <origin xyz="0 0 0" rpy="0 0 0"/>
             <geometry>
-                <mesh filename="package://monty_demo/meshes/X3plus/visual/llink2.STL"/>
-            </geometry>
-            <material name="">
-                <color rgba="0 0.7 0 1"/>
-            </material>
-        </visual>
-        <collision>
-            <origin xyz="0 0 0" rpy="0 0 0"/>
-            <geometry>
-                <mesh filename="package://monty_demo/meshes/X3plus/visual/llink2.STL"/>
+                <mesh filename="${mesh_prefix}/X3plus/visual/llink2.STL"/>
+            </geometry>
+            <material name="">
+                <color rgba="0 0.7 0 1"/>
+            </material>
+        </visual>
+        <collision>
+            <origin xyz="0 0 0" rpy="0 0 0"/>
+            <geometry>
+                <mesh filename="${mesh_prefix}/X3plus/visual/llink2.STL"/>
             </geometry>
         </collision>
@@ -463,14 +471,14 @@
             <origin xyz="0 0 0" rpy="0 0 0"/>
             <geometry>
-                <mesh filename="package://monty_demo/meshes/X3plus/visual/llink3.STL"/>
-            </geometry>
-            <material name="">
-                <color rgba="0 0.7 0 1"/>
-            </material>
-        </visual>
-        <collision>
-            <origin xyz="0 0 0" rpy="0 0 0"/>
-            <geometry>
-                <mesh filename="package://monty_demo/meshes/X3plus/visual/llink3.STL"/>
+                <mesh filename="${mesh_prefix}/X3plus/visual/llink3.STL"/>
+            </geometry>
+            <material name="">
+                <color rgba="0 0.7 0 1"/>
+            </material>
+        </visual>
+        <collision>
+            <origin xyz="0 0 0" rpy="0 0 0"/>
+            <geometry>
+                <mesh filename="${mesh_prefix}/X3plus/visual/llink3.STL"/>
             </geometry>
         </collision>
@@ -493,5 +501,5 @@
             <origin xyz="0 0 0" rpy="0 0 0"/>
             <geometry>
-                <mesh filename="package://monty_demo/meshes/sensor/visual/mono_link.STL"/>
+                <mesh filename="${mesh_prefix}/sensor/visual/mono_link.STL"/>
             </geometry>
             <material name="">
@@ -502,5 +510,5 @@
             <origin xyz="0 0 0" rpy="0 0 0"/>
             <geometry>
-                <mesh filename="package://monty_demo/meshes/sensor/collision/mono_link.STL"/>
+                <mesh filename="${mesh_prefix}/sensor/collision/mono_link.STL"/>
             </geometry>
         </collision>

Commit message: the pick and place are successful

File: docker_all/components/ros2_comp/app/monty_demo/x3plus_robot/urdf/x3plus.urdf.xacro (robot description, xacro)
@@ -519,4 +519,45 @@
         <child link="mono_link"/>
     </joint>
+    <!-- Tire/track collision volumes (collision-only, no visual).
+         Box dimensions are conservative estimates of the X3plus tracks
+         derived from: _BASE_COLL_Y_HALF=0.15, _BASE_COLL_X=(-0.13,0.07)
+         in x3plus_5dof_planner.py, padded for safety.
+         In base_link frame: ground is at z=-0.076, base bottom at z~0. -->
+    <link name="right_track_link">
+        <inertial>
+            <origin xyz="0 0 0" rpy="0 0 0"/>
+            <mass value="0.01"/>
+            <inertia ixx="1e-6" ixy="0" ixz="0" iyy="1e-6" iyz="0" izz="1e-6"/>
+        </inertial>
+        <collision>
+            <origin xyz="0 0 0" rpy="0 0 0"/>
+            <geometry>
+                <box size="0.28 0.06 0.08"/>
+            </geometry>
+        </collision>
+    </link>
+    <joint name="right_track_joint" type="fixed">
+        <origin xyz="-0.02 -0.13 -0.038" rpy="0 0 0"/>
+        <parent link="base_link"/>
+        <child link="right_track_link"/>
+    </joint>
+    <link name="left_track_link">
+        <inertial>
+            <origin xyz="0 0 0" rpy="0 0 0"/>
+            <mass value="0.01"/>
+            <inertia ixx="1e-6" ixy="0" ixz="0" iyy="1e-6" iyz="0" izz="1e-6"/>
+        </inertial>
+        <collision>
+            <origin xyz="0 0 0" rpy="0 0 0"/>
+            <geometry>
+                <box size="0.28 0.06 0.08"/>
+            </geometry>
+        </collision>
+    </link>
+    <joint name="left_track_joint" type="fixed">
+        <origin xyz="-0.02 0.13 -0.038" rpy="0 0 0"/>
+        <parent link="base_link"/>
+        <child link="left_track_link"/>
+    </joint>
     <xacro:if value="${include_ros2_control}">
         <xacro:include filename="ros2_control_topic.xacro"/>
